File: CC_PCB_V1.kicad_pcb (KiCad board)
At the start: 2 copper layers, 104.2 x 144.9 mm, 14 parts, among them J1 Screw_Terminal_01x07, J2 Antenna_Conn_02x04_Odd_Even, J3 USB1130-15-A_REVA, J5 Relay_Conn_01x06, U1 Pico, U2 LM337_TO3

Commit message: Created Gerber file
Routing:
- net GP6: track 77.6 -> 74.2 mm
- net GP4: track 78.1 -> 80.0 mm
- net GP7: track 66.1 -> 67.3 mm
Changed lines of the file:
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@@
     (thickness 1.6)
     (drawings 29)
-    (tracks 137)
+    (tracks 142)
     (zones 0)
     (modules 14)
@@
       (usegerberattributes true)
       (usegerberadvancedattributes true)
-      (creategerberjobfile true)
+      (creategerberjobfile false)
       (excludeedgelayer true)
       (linewidth 0.100000)
@@
       (effects (font (size 1 1) (thickness 0.15)))
     )
-    (fp_text user %R (at 0.3 0) (layer F.Fab)
-      (effects (font (size 1 1) (thickness 0.15)))
-    )
     (fp_circle (center 0 0) (end 3 0) (layer Cmts.User) (width 0.15))
     (fp_circle (center 0 0) (end 3.25 0) (layer F.CrtYd) (width 0.05))
+    (fp_text user %R (at 0.3 0) (layer F.Fab)
+      (effects (font (size 1 1) (thickness 0.15)))
+    )
     (pad 1 np_thru_hole circle (at 0 0) (size 3 3) (drill 3) (layers *.Cu *.Mask))
   )
@@
       (effects (font (size 1 1) (thickness 0.15)))
     )
-    (fp_text user %R (at 0.3 0) (layer F.Fab)
-      (effects (font (size 1 1) (thickness 0.15)))
-    )
     (fp_circle (center 0 0) (end 3 0) (layer Cmts.User) (width 0.15))
     (fp_circle (center 0 0) (end 3.25 0) (layer F.CrtYd) (width 0.05))
+    (fp_text user %R (at 0.3 0) (layer F.Fab)
+      (effects (font (size 1 1) (thickness 0.15)))
+    )
     (pad 1 np_thru_hole circle (at 0 0) (size 3 3) (drill 3) (layers *.Cu *.Mask))
   )
@@
       (effects (font (size 1 1) (thickness 0.15)))
     )
-    (fp_text user %R (at 0.3 0) (layer F.Fab)
-      (effects (font (size 1 1) (thickness 0.15)))
-    )
     (fp_circle (center 0 0) (end 3 0) (layer Cmts.User) (width 0.15))
     (fp_circle (center 0 0) (end 3.25 0) (layer F.CrtYd) (width 0.05))
+    (fp_text user %R (at 0.3 0) (layer F.Fab)
+      (effects (font (size 1 1) (thickness 0.15)))
+    )
     (pad 1 np_thru_hole circle (at 0 0) (size 3 3) (drill 3) (layers *.Cu *.Mask))
   )
@@
       (effects (font (size 1 1) (thickness 0.15)))
     )
-    (fp_text user %R (at 0 0) (layer F.Fab)
-      (effects (font (size 1 1) (thickness 0.15)))
-    )
     (fp_circle (center 0 0) (end 3 0) (layer Cmts.User) (width 0.15))
     (fp_circle (center 0 0) (end 3.25 0) (layer F.CrtYd) (width 0.05))
+    (fp_text user %R (at 0 0) (layer F.Fab)
+      (effects (font (size 1 1) (thickness 0.15)))
+    )
     (pad 1 np_thru_hole circle (at 0 0) (size 3 3) (drill 3) (layers *.Cu *.Mask))
   )
@@
   (segment (start 117.6 65.976485) (end 117.725 65.851485) (width 0.25) (layer F.Cu) (net 3))
   (segment (start 117.6 87.919998) (end 117.6 65.976485) (width 0.25) (layer F.Cu) (net 3))
-  (segment (start 117.725 65.851485) (end 122 61.576485) (width 0.25) (layer B.Cu) (net 3))
-  (segment (start 122 54.18) (end 128.11 48.07) (width 0.25) (layer B.Cu) (net 3))
-  (segment (start 122 61.576485) (end 122 54.18) (width 0.25) (layer B.Cu) (net 3))
-  (segment (start 128.11 58.23) (end 126.77 58.23) (width 0.25) (layer B.Cu) (net 4))
+  (segment (start 122 61.576485) (end 117.725 65.851485) (width 0.25) (layer B.Cu) (net 3))
+  (segment (start 122 51) (end 122 61.576485) (width 0.25) (layer B.Cu) (net 3))
+  (segment (start 124.93 48.07) (end 122 51) (width 0.25) (layer B.Cu) (net 3))
+  (segment (start 128.11 48.07) (end 124.93 48.07) (width 0.25) (layer B.Cu) (net 3))
   (via (at 117.8 93.8) (size 0.8) (drill 0.4) (layers F.Cu B.Cu) (net 4))
-  (segment (start 117.8 67.2) (end 117.8 93.8) (width 0.25) (layer B.Cu) (net 4))
-  (segment (start 126.77 58.23) (end 117.8 67.2) (width 0.25) (layer B.Cu) (net 4))
   (segment (start 101.6 110) (end 99 110) (width 0.25) (layer F.Cu) (net 4))
   (segment (start 117.8 93.8) (end 101.6 110) (width 0.25) (layer F.Cu) (net 4))
+  (segment (start 124.77 60.23) (end 117.8 67.2) (width 0.25) (layer B.Cu) (net 4))
+  (segment (start 124.77 58.23) (end 124.77 60.23) (width 0.25) (layer B.Cu) (net 4))
+  (segment (start 117.8 67.2) (end 117.8 93.8) (width 0.25) (layer B.Cu) (net 4))
+  (segment (start 128.11 58.23) (end 124.77 58.23) (width 0.25) (layer B.Cu) (net 4))
   (segment (start 128.11 55.69) (end 124.29 55.69) (width 0.25) (layer F.Cu) (net 5))
-  (via (at 116 54.2) (size 0.8) (drill 0.4) (layers F.Cu B.Cu) (net 5))
-  (segment (start 122.8 54.2) (end 116 54.2) (width 0.25) (layer F.Cu) (net 5))
   (segment (start 124.29 55.69) (end 122.8 54.2) (width 0.25) (layer F.Cu) (net 5))
   (segment (start 116 95) (end 99 112) (width 0.25) (layer B.Cu) (net 5))
-  (segment (start 116 54.2) (end 116 95) (width 0.25) (layer B.Cu) (net 5))
+  (via (at 116.012653 59.987347) (size 0.8) (drill 0.4) (layers F.Cu B.Cu) (net 5))
+  (segment (start 121.8 54.2) (end 116.012653 59.987347) (width 0.25) (layer F.Cu) (net 5))
+  (segment (start 122.8 54.2) (end 121.8 54.2) (width 0.25) (layer F.Cu) (net 5))
+  (segment (start 116 60.565685) (end 116 95) (width 0.25) (layer B.Cu) (net 5))
+  (segment (start 116.012653 60.553032) (end 116 60.565685) (width 0.25) (layer B.Cu) (net 5))
+  (segment (start 116.012653 59.987347) (end 116.012653 60.553032) (width 0.25) (layer B.Cu) (net 5))
   (segment (start 128.11 81.09) (end 129.49 81.09) (width 0.25) (layer F.Cu) (net 6))
   (segment (start 129.49 81.09) (end 129.8 81.4) (width 0.25) (layer F.Cu) (net 6))
@@
   (segment (start 103.5 140) (end 90.79 140) (width 0.25) (layer F.Cu) (net 8))
   (segment (start 87.695 143.095) (end 83.5 147.29) (width 0.25) (layer F.Cu) (net 8))
-  (segment (start 87.895 53.105) (end 87.895 142.895) (width 0.25) (layer F.Cu) (net 8) (status 1000000))
-  (segment (start 97 44) (end 87.895 53.105) (width 0.25) (layer F.Cu) (net 8) (status 1000000))
-  (segment (start 103 44) (end 97 44) (width 0.25) (layer F.Cu) (net 8) (status 1000000))
+  (segment (start 87.895 53.105) (end 87.895 142.895) (width 0.25) (layer F.Cu) (net 8))
+  (segment (start 97 44) (end 87.895 53.105) (width 0.25) (layer F.Cu) (net 8))
+  (segment (start 103 44) (end 97 44) (width 0.25) (layer F.Cu) (net 8))
   (segment (start 87.895 142.895) (end 87.695 143.095) (width 0.25) (layer F.Cu) (net 8))
   (segment (start 90.79 140) (end 87.895 142.895) (width 0.25) (layer F.Cu) (net 8))
